File: kicad/picoarduino.kicad_sch (KiCad schematic)
At the start: 6 parts, among them J1 Conn_02x03_Odd_Even, M1 Module_RaspberryPi_PicoW_Comb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, SW1 Switch_Tactile_Omron, U1 4053

Commit message: Schematic and PCB
Parts:
- removed XA1: Arduino_Uno_Shield, symbol arduino:Arduino_Uno_Shield
- added A1: Arduino_Leonardo, Module:Arduino_UNO_R3, symbol MCU_Module:Arduino_Leonardo
- added C2, C3: 1uF, Capacitor_SMD:C_1206_3216Metric_Pad1.33x1.80mm_HandSolder, symbol Device:C
- added D1, D2: ~, Diode_SMD:D_SMB, symbol Device:D
- added H1, H2, H3, H4: MountingHole, MountingHole:MountingHole_3.2mm_M3_DIN965, symbol Mechanical:MountingHole
- added J2: Conn_01x03_Pin, Connector_PinHeader_2.54mm:PinHeader_1x03_P2.54mm_Horizontal, symbol Connector:Conn_01x03_Pin
- added J3: Barrel_Jack_Switch, Connector_BarrelJack:BarrelJack_Horizontal, symbol Connector:Barrel_Jack_Switch
- added U2: TLV1117-5.0, Package_TO_SOT_SMD:SOT-223-3_TabPin2, symbol Regulator_Linear:LM1117MP-5.0
- C1: value C -> 100nF; footprint (none) -> Capacitor_SMD:C_1206_3216Metric_Pad1.33x1.80mm_HandSolder
- J1: footprint (none) -> Connector_PinHeader_2.54mm:PinHeader_2x03_P2.54mm_Vertical
- M1: footprint fab:RaspberryPi_PicoW_Combined -> Library:RaspberryPi_Pico
- SW1: footprint fab:Button_Omron_B3SN_6.0x6.0mm -> Library:Button_Omron_B3SN_6.0x6.0mm
- U1: value 4053 -> SN74LV4053ADR; footprint (none) -> Package_SO:SOIC-16_3.9x9.9mm_P1.27mm; MPN (none) -> SN74LV4053ADR
Connections:
- net at U1.1 (Y1): now also A1.12 (A3)
- net GP22: now reaches U1.10 (B)
- net GP22: now also M1.29 (GP22), U1.11 (A), U1.9 (C)
- net at U1.12 (X0): now also A1.9 (A0)
- net at U1.13 (X1): now also A1.10 (A1)
- net at U1.14 (X): now also M1.34 (GP28)
- net at U1.15 (Y): now also M1.32 (GP27)
- net VDD: now reaches U1.16 (VDD)
- net VDD: now also C1.1, J1.2 (Pin_2), M1.36 (3V3_OUT), A1.2 (IOREF), A1.4 (3V3)
- net at U1.2 (Y0): now also A1.11 (A2)
- net at U1.3 (Z1): now also A1.14 (A5)
- net at U1.4 (Z): now also M1.31 (GP26)
- net at U1.5 (Z0): now also A1.13 (A4)
- net GND: now reaches U1.6 (Inh)
- net GND: now also C1.2, J1.6 (Pin_6), M1.13 (GND), M1.18 (GND), M1.23 (GND), M1.28 (GND), M1.3 (GND), M1.33 (GND), M1.38 (GND), M1.42 (GND), M1.8 (GND), SW1.2, U1.7 (VEE), U1.8 (VSS), A1.29 (GND), A1.6 (GND), A1.7 (GND), C2.2, C3.2, J2.2 (Pin_2), J3.2, J3.3, U2.1 (GND)
- net nRESET: now reaches SW1.1
- net nRESET: now also M1.30 (RUN), A1.3 (~{RESET})
- net GP0: now reaches M1.1 (GP0)
- net GP0: now also A1.16 (D1/TX)
- net GP7: now reaches M1.10 (GP7)
- net GP7: now also A1.20 (D5)
- net GP8: now reaches M1.11 (GP8)
- net GP8: now also A1.21 (D6)
- net GP9: now reaches M1.12 (GP9)
- net GP9: now also A1.22 (D7)
- net GP10: now reaches M1.14 (GP10)
- net GP10: now also J1.3 (Pin_3)
- net GP11: now reaches M1.15 (GP11)
- net GP11: now also J1.4 (Pin_4)
- net GP12: now reaches M1.16 (GP12)
- net GP12: now also J1.1 (Pin_1)
- net GP13: now reaches M1.17 (GP13)
- net GP13: now also J1.5 (Pin_5)
- net GP14: now reaches M1.19 (GP14)
- net GP1: now reaches M1.2 (GP1)
- net GP1: now also A1.15 (D0/RX)
- net GP15: now reaches M1.20 (GP15)
- net GP16: now reaches M1.21 (GP16)
- net GP16: now also A1.27 (D12)
- net GP17: now reaches M1.22 (GP17)
- net GP17: now also A1.25 (D10)
- net GP18: now reaches M1.24 (GP18)
- net GP18: now also A1.28 (D13)
- net GP19: now reaches M1.25 (GP19)
- net GP19: now also A1.26 (D11)
- net GP20: now reaches M1.26 (GP20)
- net GP20: now also A1.31 (SDA/D2)
- net GP21: now reaches M1.27 (GP21)
- net GP21: now also A1.32 (SCL/D3)
- net VREF: now reaches M1.35 (ADC_VREF)
- net VREF: now also A1.30 (AREF)
- net +5V: now reaches M1.39 (VSYS)
- net +5V: now also A1.5 (+5V), D2.1 (K)
- net GP2: now reaches M1.4 (GP2)
- net GP2: now also A1.23 (D8)
- net GP3: now reaches M1.5 (GP3)
- net GP3: now also A1.24 (D9)
- net GP4: now reaches M1.6 (GP4)
- net GP4: now also A1.17 (D2/SDA)
- net GP5: now reaches M1.7 (GP5)
- net GP5: now also A1.18 (D3/SCL)
- net GP6: now reaches M1.9 (GP6)
- net GP6: now also A1.19 (D4)
- new net: C3.1, D2.2 (A), U2.2 (VO)
- new net: D1.2 (A), J3.1
- new net SWCLK: J2.3 (Pin_3), M1.41 (SWCLK)
- new net SWDIO: J2.1 (Pin_1), M1.43 (SWDIO)
- new net VIN: A1.8 (VIN), C2.1, D1.1 (K), U2.3 (VI)
- no-connect marks 0 -> 1
Other:
- moved on the sheet: C1, SW1, U1

Commit message: Bill of materials
Parts:
- C1: MPN (none) -> CL31B104KBCNNNC; Manufacturer (none) -> Samsung Electro-mechanics; POFarnell (none) -> 3013521; POMouser (none) -> 187-CL31B104KBCNNNC
- C2: value 1uF -> 10uF; symbol Device:C -> Device:C_Polarized; MPN (none) -> TAJB106M025RNJ; Manufacturer (none) -> KYOCERA AVX; POFarnell (none) -> 2852729; POMouser (none) -> 581-TAJB106M025RNJ
- C3: value 1uF -> 10uF; symbol Device:C -> Device:C_Polarized
- D2: MPN (none) -> STPS1L30U; Manufacturer (none) -> STMicroelectronics; POFarnell (none) -> 1467550; POMouser (none) -> 511-STPS1L30U
- J3: MPN (none) -> DCJ235-05-A-K1-K; Manufacturer (none) -> GCT; POFarnell (none) -> 3873896; POMouser (none) -> 640-DCJ235-05-A-K1-K
- SW1: MPN (none) -> PTS526SM20SMTR21; Manufacturer (none) -> C&K; POFarnell (none) -> 3941499; POMouser (none) -> 611-PTS526SM20S21LFS
- U1: MPN SN74LV4053ADR -> 74LV4053D,118; Manufacturer (none) -> Nexperia; POFarnell (none) -> 3441376; POMouser (none) -> 771-LV4053D118
- U2: MPN (none) -> TLV1117-50IDCYR; Manufacturer (none) -> Texas Instruments; POFarnell (none) -> 3122345; POMouser (none) -> 595-TLV1117-50IDCYR
Connections:
- net GND: no longer C2.2, C3.2
- net VIN: no longer C2.1
- net at D2.2 (A), U2.2 (VO): no longer C3.1
